File: schematc-io.kicad_sch (KiCad schematic)
At the start: 0 parts

Commit message: Update project structure to fit its name
Parts:
- added C27: 4n7, symbol Device:C
- added C7: 100n, symbol Device:C
- added D2, D3, D4: LED, symbol Device:LED
- added D5: SP0502BAJT, Package_TO_SOT_SMD:SOT-323_SC-70, symbol Power_Protection:SP0502BAJT
- added R14, R16: 100, symbol Device:R
- added R17, R18: 60, symbol Device:R
- added R17: 270, symbol Device:R
- added R2, R3, R4: 1k, symbol Device:R
- added U3: SN65HVD232, Package_SO:SOIC-8_3.9x4.9mm_P1.27mm, symbol Interface_CAN_LIN:SN65HVD232
- added U7: PC817, Package_DIP:DIP-4_W7.62mm, symbol Isolator:PC817
- added U8: TLP250, Package_DIP:DIP-8_W7.62mm, symbol Driver_FET:TLP250
Connections:
- new net: D4.1 (K), R4.1
- new net: C27.1, R17.1, R18.1
- new net: D3.1 (K), R2.1
- new net: R14.2, U8.2 (A)
- new net: D2.1 (K), R3.1
- new net: R16.2, U7.1
- new net +12V: R17.1, U8.8 (VCC)
- new net +3.3V: C7.1, D4.2 (A), U3.3 (VCC)
- new net CANH: D5.1 (K), R17.2, U3.7 (CANH)
- new net CANL: D5.2 (K), R18.2, U3.6 (CANL)
- new net CAN_RX: U3.1 (D)
- new net CAN_TX: U3.4 (R)
- new net FAN_1_PWM: U8.6 (VO)
- new net FAN_2_PWM: U8.7 (VO)
- new net FAN_PWM_MCU: R14.1
- new net GND: C27.2, C7.2, D5.3 (A), R2.2, R3.2, R4.2, U3.2 (GND), U7.2, U7.3, U8.3 (C), U8.5 (VEE)
- new net LED_CAN_STATUS: D3.2 (A)
- new net LED_MCU_STATUS: D2.2 (A)
- new net PURGE_VALVE: R17.2, U7.4
- new net PURGE_VALVE_MCU: R16.1
Other:
- note added: "CAN Transceiver"
- note added: "Fan drivers"
- note added: "If = ( Vdd - Vf ) / Rf = ( 3.3V - 0.7V ) / 100ohm = 26mA"
- note added: "Purge valve driver"
- note added: "Rc > [ ( Vcc - VCEsat ) / ( CTR x If ) ] = [ ( 5V - 0V ) / ( 80% x 26mA ) ] = 240.38Ω"
- note added: "Rf > [ ( Vdd - Vf ) / ( 80% x Irating ) ] = [ ( 3.3V - 0.7V ) / ( 80% x 40mA ) ] = 81.25Ω"
- note added: "Signal diodes"
- note added: "TODO: 12V?"
- note added: "TODO: add calculations"
- note added: "TODO: verify circuit"
- note added: "Termination node (resistors and capacitor) may be omitted during assembly if not required."
- company: (none) -> Hydrogreen Pollub
- title: (none) -> Motor driver unit
