File: schematc-io.kicad_sch (KiCad schematic)
At the start: 17 parts, among them U3 SN65HVD232, U7 PC817, U8 TLP250

Commit message: Add power stages
Valve, power supplay, fan
Parts:
- removed R14: 100, symbol Device:R
- removed U8: TLP250, Package_DIP:DIP-8_W7.62mm, symbol Driver_FET:TLP250
- added C31: 20n, symbol Device:C
- added D8: 1N5819, Diode_THT:D_DO-41_SOD81_P10.16mm_Horizontal, symbol Diode:1N5819
- added Q1: DMP10H400SK3-13, DMP10H400SK313, symbol p-mosfet:DMP10H400SK3-13
- added Q2, Q5: IRLZ44N, Package_TO_SOT_THT:TO-220-3_Vertical, symbol Transistor_FET:IRLZ44N
- added Q3, Q4: 2N3904, Package_TO_SOT_THT:TO-92_Inline, symbol Transistor_BJT:2N3904
- added R26: 100R 0,5W, symbol Device:R
- added R27, R30, R37: 1k, symbol Device:R
- added R28, R31, R33: 100, symbol Device:R
- added R29, R32: 10k, symbol Device:R
- added R34: 0, symbol Device:R
- added U8: PC817, Package_DIP:DIP-4_W7.62mm, symbol Isolator:PC817
- R17: value 270 -> 1k
Connections:
- net +12V: now also D8.1 (K), Q1.3 (S), R27.1, R30.1, R37.1
- net GND: now also Q2.3 (S), Q3.1 (E), Q4.1 (E), Q5.3 (S), R26.2, R29.2, R32.2, R34.2, U8.2, U8.3
- net PURGE_VALVE: no longer names the net of R17.2, U7.4
- net PURGE_VALVE: now also Q3.2 (B)
- new net: Q3.3 (C), R27.2, R28.1
- new net: Q2.1 (G), R28.2, R29.1
- new net: Q4.2 (B), R37.2, U8.4
- new net: Q4.3 (C), R30.2, R31.1
- new net: C31.2, R26.1
- new net: Q5.1 (G), R31.2, R32.1
- new net: R33.2, U8.1
- new net +12: Q1.2 (D)
- new net FAN_GND: Q5.2 (D), R34.1
- new net FAN_ON_MCU: R33.1
- new net PURGE_VALVE_GND: C31.1, D8.2 (A), Q2.2 (D)
Other:
- note added: "Charging"
- note added: "Fan"
- note removed: "Fan drivers"
- note removed: "If = ( Vdd - Vf ) / Rf = ( 3.3V - 0.7V ) / 100ohm = 26mA"
- note removed: "Rc > [ ( Vcc - VCEsat ) / ( CTR x If ) ] = [ ( 5V - 0V ) / ( 80% x 26mA ) ] = 240.38Ω"
- note removed: "Rf > [ ( Vdd - Vf ) / ( 80% x Irating ) ] = [ ( 3.3V - 0.7V ) / ( 80% x 40mA ) ] = 81.25Ω"
- note removed: "TODO: add calculations"
- note removed: "TODO: verify circuit"
- moved on the sheet: R16, R17, U7

Commit message: Add tags
Edit main schema and sockets
Connections:
- net +12V: no longer Q1.3 (S)
- new net out_12V: Q1.3 (S)
Other:
- note removed: "TODO: 12V?"
- moved on the sheet: C27, C7, D5, R17, R18, U3

Commit message: Add FC voltage measure, axilary input and output
Schematic complet?
Parts:
- removed Q1: DMP10H400SK3-13, DMP10H400SK313, symbol p-mosfet:DMP10H400SK3-13
- added C27 (x3): 4n7, symbol Device:C
- added C32: 20n, symbol Device:C
- added D9: 1N5819, Diode_THT:D_DO-41_SOD81_P10.16mm_Horizontal, symbol Diode:1N5819
- added IC1: AD8544ARUZ-REEL, SOP65P640X120-14N, symbol ad8544:AD8544ARUZ-REEL
- added Q6: 2N3904, lib:SOT65P220X100-3N, symbol Transistor_BJT:2N3904
- added Q7: sir186, lib:SI7141DPT1GE3, symbol Transistor_FET:IRLZ44N
- added R18, R2, R43: 10k, symbol Device:R
- added R18: 150k, symbol Device:R
- added R2: 560k, symbol Device:R
- added R39, R42: 100, symbol Device:R
- added R40, R41: 1k, symbol Device:R
- added R44: 100R 0,5W, symbol Device:R
- added U9: PC817, Package_DIP:DIP-4_W7.62mm, symbol Isolator:PC817
- Q2, Q5: value IRLZ44N -> sir186; footprint Package_TO_SOT_THT:TO-220-3_Vertical -> lib:SI7141DPT1GE3
- Q3, Q4: footprint Package_TO_SOT_THT:TO-92_Inline -> lib:SOT65P220X100-3N
Connections:
- net +12V: now also D9.1 (K), R40.1, R41.1
- net +3.3V: now also IC1.4 (V+)
- net GND: now also C27.1, C27.1, C27.2, IC1.11 (V-), Q6.1 (E), Q7.3 (S), R18.1, R2.2, R2.2, R43.2, R44.2, U9.2, U9.3
- new net: IC1.12 (+IN_D), R18.1, R18.2
- new net: Q6.3 (C), R41.2, R42.1
- new net: Q7.1 (G), R42.2, R43.1
- new net: R39.2, U9.1
- new net: Q6.2 (B), R40.2, U9.4
- new net: C32.2, R44.1
- new net A_Input: IC1.5 (+IN_B), R2.1
- new net Analog_MCU: C27.1, IC1.6 (-IN_B), IC1.7 (OUT_B)
- new net FC_Voltage_MCU: C27.2, IC1.13 (-IN_D), IC1.14 (OUT_D)
- new net PWM_Out: C32.1, D9.2 (A), Q7.2 (D)
- new net PWM_Output_MCU: R39.1
- new net SC_V: R18.2
- new net Temp_MCU: C27.2, IC1.1 (OUT_A), IC1.2 (-IN_A)
- new net Temp_sensor: IC1.3 (+IN_A), R2.1
- no-connect marks 0 -> 3
Other:
- note added: "Amplifire"
- note added: "Axilary driver"
- note added: "Fan driver"
- note removed: "Charging"
- note removed: "Fan"
- title: Motor driver unit -> Fuel Cell Control Unit  (FCCU)
- moved on the sheet: C27, C7, D2, D3, D4, D5, Q4, Q5, R17, R18, R2, R3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

Commit message: First pcb, change fan conector
Parts:
- removed R34: 0, symbol Device:R
- added C7: 100n, Capacitor_SMD:C_1206_3216Metric, symbol Device:C
- C27, C31, C32, C7: footprint (none) -> Capacitor_SMD:C_1206_3216Metric
- D2, D3, D4: footprint (none) -> Diode_SMD:D_1206_3216Metric
- IC1: footprint SOP65P640X120-14N -> lib:SOP65P640X120-14N
- R16, R17: footprint (none) -> Resistor_SMD:R_1206_3216Metric
- R18, R2, R27, R28, R29, R3, R30, R31, R32, R33, R37, R39, R4, R40, R41, R42, R43: footprint (none) -> LED_SMD:LED_1206_3216Metric
- R26, R44: footprint (none) -> Resistor_SMD:R_2512_6332Metric
Connections:
- net +3.3V: now also C7.1
- net GND: now also C7.2

Commit message: Change FC connector to 10pin & ideal diode sircuit
Parts:
- IC1: footprint lib:SOP65P640X120-14N -> library:SOP65P640X120-14N
- Q2, Q5, Q7: footprint lib:SI7141DPT1GE3 -> library:SI7141DPT1GE3
- Q3, Q4, Q6: footprint lib:SOT65P220X100-3N -> library:SOT65P220X100-3N
Connections:
- net PWM_Out renamed Main_Valve
- net PWM_Output_MCU renamed Main_Valve_MCU
Changed lines of the file:
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@@
     (effects (font (size 1.27 1.27)) (justify right))
   )
-  (hierarchical_label "PWM_Out" (shape output) (at 256.921 89.662 0) (fields_autoplaced)
+  (hierarchical_label "Main_Valve" (shape output) (at 256.921 89.662 0) (fields_autoplaced)
     (effects (font (size 1.27 1.27)) (justify left))
   )
@@
     (effects (font (size 1.27 1.27)) (justify left))
   )
-  (hierarchical_label "PWM_Output_MCU" (shape input) (at 180.721 99.822 180) (fields_autoplaced)
+  (hierarchical_label "Main_Valve_MCU" (shape input) (at 180.721 99.822 180) (fields_autoplaced)
     (effects (font (size 1.27 1.27)) (justify right))
   )
@@
       (effects (font (size 1.27 1.27)) (justify left))
     )
-    (property "Footprint" "lib:SOT65P220X100-3N" (at 228.346 149.098 0)
+    (property "Footprint" "library:SOT65P220X100-3N" (at 228.346 149.098 0)
       (effects (font (size 1.27 1.27) italic) (justify left) hide)
     )
@@
       (effects (font (size 1.27 1.27)) (justify left))
     )
-    (property "Footprint" "lib:SOT65P220X100-3N" (at 230.251 101.727 0)
+    (property "Footprint" "library:SOT65P220X100-3N" (at 230.251 101.727 0)
       (effects (font (size 1.27 1.27) italic) (justify left) hide)
     )
@@
       (effects (font (size 1.27 1.27)) (justify left))
     )
-    (property "Footprint" "lib:SOT65P220X100-3N" (at 233.68 55.245 0)
+    (property "Footprint" "library:SOT65P220X100-3N" (at 233.68 55.245 0)
       (effects (font (size 1.27 1.27) italic) (justify left) hide)
     )
@@
       (effects (font (size 1.27 1.27)) (justify left))
     )
-    (property "Footprint" "lib:SI7141DPT1GE3" (at 252.73 50.165 0)
+    (property "Footprint" "library:SI7141DPT1GE3" (at 252.73 50.165 0)
       (effects (font (size 1.27 1.27) italic) (justify left) hide)
     )
@@
       (effects (font (size 1.27 1.27)) (justify left))
     )
-    (property "Footprint" "lib:SI7141DPT1GE3" (at 249.301 96.647 0)
+    (property "Footprint" "library:SI7141DPT1GE3" (at 249.301 96.647 0)
       (effects (font (size 1.27 1.27) italic) (justify left) hide)
     )
@@
       (effects (font (size 1.27 1.27)))
     )
-    (property "Footprint" "lib:SOP65P640X120-14N" (at 65.532 201.854 0)
+    (property "Footprint" "library:SOP65P640X120-14N" (at 65.532 201.854 0)
       (effects (font (size 1.27 1.27)) (justify left top) hide)
     )
@@
       (effects (font (size 1.27 1.27)) (justify left))
     )
-    (property "Footprint" "lib:SI7141DPT1GE3" (at 247.396 144.018 0)
+    (property "Footprint" "library:SI7141DPT1GE3" (at 247.396 144.018 0)
       (effects (font (size 1.27 1.27) italic) (justify left) hide)
     )

Commit message: Complate frist version
Parts:
- removed C32: 20n, Capacitor_SMD:C_1206_3216Metric, symbol Device:C
- removed D9: 1N5819, Diode_THT:D_DO-41_SOD81_P10.16mm_Horizontal, symbol Diode:1N5819
- removed Q2, Q5, Q7: sir186, library:SI7141DPT1GE3, symbol Transistor_FET:IRLZ44N
- added C37: 20n, Capacitor_SMD:C_1206_3216Metric, symbol Device:C
- added D10: 1N5819, Diode_THT:D_DO-41_SOD81_P10.16mm_Horizontal, symbol Diode:1N5819
- added Q1, Q2, Q5: SIR186LDP-T1-RE3, SI7141DPT1GE3, symbol sir186 ldp-t1-re3 mosfet 60v:SIR186LDP-T1-RE3
Connections:
- net +12V: now also D10.1 (K)
- net FAN_GND: now also Q2.10 (D_6), Q2.11 (D_7), Q2.5 (D_1), Q2.6 (D_2), Q2.7 (D_3), Q2.8 (D_4), Q2.9 (D_5)
- net GND: now also Q1.1 (S_1), Q1.2 (S_2), Q1.3 (S_3), Q2.1 (S_1), Q2.2 (S_2), Q2.3 (S_3), Q5.1 (S_1), Q5.2 (S_2), Q5.3 (S_3)
- net Main_Valve: now also C37.1, D10.2 (A), Q5.10 (D_6), Q5.11 (D_7), Q5.5 (D_1), Q5.6 (D_2), Q5.7 (D_3), Q5.8 (D_4), Q5.9 (D_5)
- net at R28.2, R29.1: now also Q1.4 (G)
- net at R42.2, R43.1: now also Q5.4 (G)
- net at R31.2, R32.1: now also Q2.4 (G)
- net at R44.1: now also C37.2
- net PURGE_VALVE_GND renamed PURGE_VALVE
- net PURGE_VALVE: now also Q1.10 (D_6), Q1.11 (D_7), Q1.5 (D_1), Q1.6 (D_2), Q1.7 (D_3), Q1.8 (D_4), Q1.9 (D_5)
Other:
- moved on the sheet: C31, D8, Q3, Q6, R16, R17, R26, R27, R28, R29, R39, R40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

Commit message: porawa library
Connections:
- net SC_V renamed FC_V
Other:
- note added: "Voltage follower"
- note removed: "Amplifire"
- moved on the sheet: C27, C7, IC1, R18, R2

Commit message: Edit main
Parts:
- removed Q1, Q2, Q5: SIR186LDP-T1-RE3, SI7141DPT1GE3, symbol sir186 ldp-t1-re3 mosfet 60v:SIR186LDP-T1-RE3
- removed Q3, Q4, Q6: 2N3904, library:SOT65P220X100-3N, symbol Transistor_BJT:2N3904
- removed R29, R32, R43: 10k, LED_SMD:LED_1206_3216Metric, symbol Device:R
- removed R30, R37, R40, R41: 1k, LED_SMD:LED_1206_3216Metric, symbol Device:R
- removed R31, R33, R39, R42: 100, LED_SMD:LED_1206_3216Metric, symbol Device:R
- removed U7, U8, U9: PC817, Package_DIP:DIP-4_W7.62mm, symbol Isolator:PC817
- added MOSFET1, MOSFET2: PMPB15XP_115, DFN2020MD-6_SOT1220_NEX, symbol mosfet logic:PMPB15XP_115
- added R2 (x2): 10k, LED_SMD:LED_1206_3216Metric, symbol Device:R
- added TP1, TP2: GND, symbol Connector:TestPoint
- added TP10: I/O 2, symbol Connector:TestPoint
- added TP11: I/O 3, symbol Connector:TestPoint
- added TP12: I/O 4, symbol Connector:TestPoint
- added TP3, TP4: +12V, symbol Connector:TestPoint
- added TP5, TP6: +5V, symbol Connector:TestPoint
- added TP7, TP8: +3.3V, symbol Connector:TestPoint
- added TP9: I/O 1, symbol Connector:TestPoint
- D10: value 1N5819 -> PMEG10020
- D8: value 1N5819 -> PMEG10020; footprint Diode_THT:D_DO-41_SOD81_P10.16mm_Horizontal -> (none)
- R16: value 100 -> 1k
- R27: value 1k -> 100R; footprint LED_SMD:LED_1206_3216Metric -> Resistor_SMD:R_1206_3216Metric
- R28: value 100 -> 100R; footprint LED_SMD:LED_1206_3216Metric -> Resistor_SMD:R_1206_3216Metric
Connections:
- net +12V: now also TP3.1, TP4.1; no longer R17.1, R27.1
- net +3.3V: now also TP7.1, TP8.1
- net GND: now also R2.2, R2.2, TP1.1, TP2.1; no longer R26.2
- net PURGE_VALVE_MCU: no longer R16.1
- net at R28.1: now also TP12.1; no longer R27.2
- net I/O_4_MCU: now reaches R28.2
- net I/O_4_MCU: now also R2.1
- net I/O_2_MCU: now reaches R17.2
- net I/O_1_MCU: now reaches R16.2
- new net: R27.1, TP11.1
- new net: R16.1, TP9.1
- new net: R17.1, TP10.1
- new net +5V: TP5.1, TP6.1
- new net I/O_3_MCU: R2.1, R27.2
Other:
- note added: "Test points"
- note removed: "Fan driver"
- moved on the sheet: C27, C7, D5, IC1, R17, R18, R2, U3
