File: schematc-io.kicad_sch (KiCad schematic)
At the start: 47 parts, among them IC1 AD8544ARUZ-REEL, U3 SN65HVD232

Commit message: Valve driver
Parts:
- removed C37: 20n, Capacitor_SMD:C_1206_3216Metric, symbol Device:C
- removed D10: PMEG10020, Diode_THT:D_DO-41_SOD81_P10.16mm_Horizontal, symbol Diode:1N5819
- removed MOSFET2: PMPB15XP_115, DFN2020MD-6_SOT1220_NEX, symbol mosfet logic:PMPB15XP_115
- removed R44: 100R 0,5W, Resistor_SMD:R_2512_6332Metric, symbol Device:R
- added Q1: Q_NMOS_DGS, symbol Device:Q_NMOS_DGS
- added R18: 180R, LED_SMD:LED_1206_3216Metric, symbol Device:R
- MOSFET1: footprint DFN2020MD-6_SOT1220_NEX -> (none)
Connections:
- net GND: now also MOSFET1.4, MOSFET1.8, R26.2
- net PURGE_VALVE: now also MOSFET1.7
- net PURGE_VALVE_MCU: now also R18.2
- net at MOSFET1.3: now also R18.1
Other:
- moved on the sheet: C31, D8, MOSFET1, R26

Commit message: New pcb 1
Parts:
- removed MOSFET1: PMPB15XP_115, symbol mosfet logic:PMPB15XP_115
- added C36, C37: 20n, Capacitor_SMD:C_1206_3216Metric, symbol Device:C
- added D10, D9: PMEG10020, library:PMEG10020ELR, symbol Diode:1N5819
- added Q2, Q3: PMPB10XNX, library:PMPB15XPAX, symbol Device:Q_NMOS_DGS
- added R18 (x2): 180R, LED_SMD:LED_1206_3216Metric, symbol Device:R
- added R2 (x3): 10k, LED_SMD:LED_1206_3216Metric, symbol Device:R
- added R45, R46: 100R 0,5W, Resistor_SMD:R_2512_6332Metric, symbol Device:R
- D8: footprint (none) -> library:PMEG10020ELR
- Q1: value Q_NMOS_DGS -> PMPB10XNX; footprint (none) -> library:PMPB15XPAX
- TP10: renamed from TP9; footprint (none) -> Connector_PinSocket_2.54mm:PinSocket_1x01_P2.54mm_Vertical
- TP11: renamed from TP10; footprint (none) -> Connector_PinSocket_2.54mm:PinSocket_1x01_P2.54mm_Vertical
- TP12: renamed from TP11; footprint (none) -> Connector_PinSocket_2.54mm:PinSocket_1x01_P2.54mm_Vertical
- TP13: renamed from TP12; footprint (none) -> Connector_PinSocket_2.54mm:PinSocket_1x01_P2.54mm_Vertical
- TP2: renamed from TP1; footprint (none) -> Connector_PinSocket_2.54mm:PinSocket_1x01_P2.54mm_Vertical
- TP3: renamed from TP2; footprint (none) -> Connector_PinSocket_2.54mm:PinSocket_1x01_P2.54mm_Vertical
- TP4: renamed from TP3; footprint (none) -> Connector_PinSocket_2.54mm:PinSocket_1x01_P2.54mm_Vertical
- TP5: renamed from TP4; footprint (none) -> Connector_PinSocket_2.54mm:PinSocket_1x01_P2.54mm_Vertical
- TP6: renamed from TP5; footprint (none) -> Connector_PinSocket_2.54mm:PinSocket_1x01_P2.54mm_Vertical
- TP7: renamed from TP6; footprint (none) -> Connector_PinSocket_2.54mm:PinSocket_1x01_P2.54mm_Vertical
- TP8: renamed from TP7; footprint (none) -> Connector_PinSocket_2.54mm:PinSocket_1x01_P2.54mm_Vertical
- TP9: renamed from TP8; footprint (none) -> Connector_PinSocket_2.54mm:PinSocket_1x01_P2.54mm_Vertical
- renumbered C31 to C35, IC1 to IC2, R16 to R25, R17 to R26, R26 to R44
Connections:
- net +12V: now also D10.1 (K), D9.1 (K)
- net FAN_GND: now also C36.1, D9.2 (A), Q2.1 (D)
- net FAN_ON_MCU: now also R18.2
- net GND: now also Q1.3 (S), Q2.3 (S), Q3.3 (S), R2.2, R2.2, R2.2, R45.2, R46.2
- net Main_Valve: now also C37.1, D10.2 (A), Q3.1 (D)
- net Main_Valve_MCU: now also R18.2
- net PURGE_VALVE: now also Q1.1 (D)
- net at R18.1: now also Q1.2 (G), R2.1
- new net: C37.2, R46.1
- new net: Q2.2 (G), R18.1, R2.1
- new net: C36.2, R45.1
- new net: Q3.2 (G), R18.1, R2.1
Other:
- note added: "Fan driver"
- note added: "Valve driver"
- note removed: "Axilary driver"
- moved on the sheet: C35, D8, Q1, R18, R44

Commit message: Power stage pcb complate
Parts:
- renumbered C7 to C29, C27 to C30, C7 to C31, C27 to C32, C27 to C33, C27 to C34, D5 to D4, D3 to D5, D2 to D6, D4 to D7, R18 to R23, R18 to R24, R2 to R29, R2 to R30, R17 to R31, R18 to R32, R2 to R33, R2 to R34, R2 to R35, R3 to R36, R4 to R37, R18 to R38, R18 to R39, R18 to R40, R2 to R41, R2 to R42, R2 to R43, U3 to U5

Commit message: New pcb 2
Near complate
Changed lines of the file:
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@@
 	)
 	(junction
-		(at 30.48 40.005)
+		(at 30.48 34.29)
 		(diameter 0)
 		(color 0 0 0 0)
@@
 	)
 	(junction
-		(at 30.48 60.325)
+		(at 30.48 68.58)
 		(diameter 0)
 		(color 0 0 0 0)
@@
 	(wire
 		(pts
-			(xy 34.2392 40.005) (xy 30.48 40.005)
+			(xy 34.2392 34.29) (xy 30.48 34.29)
 		)
 		(stroke
@@
 	(wire
 		(pts
-			(xy 30.48 36.195) (xy 30.48 40.005)
+			(xy 30.48 32.385) (xy 30.48 34.29)
 		)
 		(stroke
@@
 	(wire
 		(pts
-			(xy 25.4 56.515) (xy 30.48 56.515)
+			(xy 25.4 64.77) (xy 30.48 64.77)
 		)
 		(stroke
@@
 	(wire
 		(pts
-			(xy 25.4 40.005) (xy 30.48 40.005)
+			(xy 25.4 34.29) (xy 30.48 34.29)
 		)
 		(stroke
@@
 	(wire
 		(pts
-			(xy 25.4 52.705) (xy 30.48 52.705)
+			(xy 25.4 60.96) (xy 30.48 60.96)
 		)
 		(stroke
@@
 	(wire
 		(pts
-			(xy 30.48 60.325) (xy 33.909 60.325)
+			(xy 30.48 68.58) (xy 33.909 68.58)
 		)
 		(stroke
@@
 	(wire
 		(pts
-			(xy 30.48 56.515) (xy 30.48 60.325)
+			(xy 30.48 64.77) (xy 30.48 68.58)
 		)
 		(stroke
@@
 	(wire
 		(pts
+			(xy 30.48 46.99) (xy 30.48 45.72)
+		)
+		(stroke
+			(width 0)
+			(type default)
+		)
+	)
+	(wire
+		(pts
 			(xy 131.445 47.625) (xy 131.445 55.245)
 		)
@@
 	(wire
 		(pts
-			(xy 30.48 52.705) (xy 30.48 48.895)
+			(xy 30.48 60.96) (xy 30.48 59.69)
 		)
 		(stroke
@@
 	(wire
 		(pts
+			(xy 25.4 46.99) (xy 30.48 46.99)
+		)
+		(stroke
+			(width 0)
+			(type default)
+		)
+	)
+	(wire
+		(pts
 			(xy 28.575 142.875) (xy 28.575 149.225)
 		)
@@
 		)
 	)
+	(hierarchical_label "5V"
+		(shape input)
+		(at 25.4 46.99 180)
+		(fields_autoplaced yes)
+		(effects
+			(font
+				(size 1.27 1.27)
+			)
+			(justify right)
+		)
+	)
 	(hierarchical_label "out_12V"
 		(shape input)
-		(at 34.2392 40.005 0)
+		(at 34.2392 34.29 0)
 		(fields_autoplaced yes)
 		(effects
@@
 		)
 	)
+	(hierarchical_label "FAN_IN_PWM_MCU"
+		(shape output)
+		(at 248.92 157.48 180)
+		(fields_autoplaced yes)
+		(effects
+			(font
+				(size 1.27 1.27)
+			)
+			(justify right)
+		)
+	)
 	(hierarchical_label "CANL"
 		(shape bidirectional)
@@
 	(hierarchical_label "3.3V"
 		(shape input)
-		(at 25.4 52.705 180)
+		(at 25.4 60.96 180)
 		(fields_autoplaced yes)
 		(effects
@@
 	(hierarchical_label "12V"
 		(shape input)
-		(at 25.4 40.005 180)
+		(at 25.4 34.29 180)
 		(fields_autoplaced yes)
 		(effects
@@
 		)
 	)
+	(hierarchical_label "FAN_IN_PWM"
+		(shape input)
+		(at 248.92 157.48 0)
+		(fields_autoplaced yes)
+		(effects
+			(font
+				(size 1.27 1.27)
+			)
+			(justify left)
+		)
+	)
 	(hierarchical_label "CANH"
 		(shape bidirectional)
@@
 	(hierarchical_label "GND"
 		(shape passive)
-		(at 25.4 56.515 180)
+		(at 25.4 64.77 180)
 		(fields_autoplaced yes)
 		(effects
@@
 	(symbol
 		(lib_id "power:GND")
-		(at 33.909 60.325 0)
+		(at 33.909 68.58 0)
 		(unit 1)
 		(exclude_from_sim no)
@@
 		(fields_autoplaced yes)
 		(property "Reference" "#PWR062"
-			(at 33.909 66.675 0)
+			(at 33.909 74.93 0)
 			(effects
 				(font
@@
 		)
 		(property "Value" "GND"
-			(at 33.909 64.77 0)
+			(at 33.909 73.025 0)
 			(effects
 				(font
@@
 		)
 		(property "Footprint" ""
-			(at 33.909 60.325 0)
+			(at 33.909 68.58 0)
 			(effects
 				(font
@@
 		)
 		(property "Datasheet" ""
-			(at 33.909 60.325 0)
+			(at 33.909 68.58 0)
 			(effects
 				(font
@@
 		)
 		(property "Description" ""
-			(at 33.909 60.325 0)
+			(at 33.909 68.58 0)
 			(effects
 				(font
@@
 	(symbol
 		(lib_id "power:+3.3V")
-		(at 30.48 48.895 0)
+		(at 30.48 59.69 0)
 		(unit 1)
 		(exclude_from_sim no)
@@
 		(fields_autoplaced yes)
 		(property "Reference" "#PWR060"
-			(at 30.48 52.705 0)
+			(at 30.48 63.5 0)
 			(effects
 				(font
@@
 		)
 		(property "Value" "+3.3V"
-			(at 30.48 43.815 0)
+			(at 30.48 54.61 0)
 			(effects
 				(font
@@
 		)
 		(property "Footprint" ""
-			(at 30.48 48.895 0)
+			(at 30.48 59.69 0)
 			(effects
 				(font
@@
 		)
 		(property "Datasheet" ""
-			(at 30.48 48.895 0)
+			(at 30.48 59.69 0)
 			(effects
 				(font
@@
 		)
 		(property "Description" ""
-			(at 30.48 48.895 0)
+			(at 30.48 59.69 0)
 			(effects
 				(font
@@
 	)
 	(symbol
+		(lib_id "power:+5V")
+		(at 30.48 45.72 0)
+		(unit 1)
+		(exclude_from_sim no)
+		(in_bom yes)
+		(on_board yes)
+		(dnp no)
+		(property "Reference" "#PWR092"
+			(at 30.48 49.53 0)
+			(effects
+				(font
+					(size 1.27 1.27)
+				)
+				(hide yes)
+			)
+		)
+		(property "Value" "+5V"
+			(at 30.48 41.656 0)
+			(effects
+				(font
+					(size 1.27 1.27)
+				)
+			)
+		)
+		(property "Footprint" ""
+			(at 30.48 45.72 0)
+			(effects
+				(font
+					(size 1.27 1.27)
+				)
+				(hide yes)
+			)
+		)
+		(property "Datasheet" ""
+			(at 30.48 45.72 0)
+			(effects
+				(font
+					(size 1.27 1.27)
+				)
+				(hide yes)
+			)
+		)
+		(property "Description" ""
+			(at 30.48 45.72 0)
+			(effects
+				(font
+					(size 1.27 1.27)
+				)
+				(hide yes)
+			)
+		)
+		(pin "1"
+		)
+		(instances
+			(project "schematic-main"
+				(path "/c9ad7189-d3b2-414a-9743-efd8e57cd755/e4695f4d-6fa6-4597-a598-6a2f28a255eb"
+					(reference "#PWR092")
+					(unit 1)
+				)
+			)
+		)
+	)
+	(symbol
 		(lib_id "Device:R")
 		(at 34.417 106.426 0)
@@
 	(symbol
 		(lib_id "power:+12V")
-		(at 30.48 36.195 0)
+		(at 30.48 32.385 0)
 		(unit 1)
 		(exclude_from_sim no)
@@
 		(fields_autoplaced yes)
 		(property "Reference" "#PWR059"
-			(at 30.48 40.005 0)
+			(at 30.48 36.195 0)
 			(effects
 				(font
@@
 		)
 		(property "Value" "+12V"
-			(at 30.48 31.115 0)
+			(at 30.48 27.305 0)
 			(effects
 				(font
@@
 		)
 		(property "Footprint" ""
-			(at 30.48 36.195 0)
+			(at 30.48 32.385 0)
 			(effects
 				(font
@@
 		)
 		(property "Datasheet" ""
-			(at 30.48 36.195 0)
+			(at 30.48 32.385 0)
 			(effects
 				(font
@@
 		)
 		(property "Description" ""
-			(at 30.48 36.195 0)
+			(at 30.48 32.385 0)
 			(effects
 				(font
@@
 	(symbol
 		(lib_id "power:GND")
-		(at 30.48 60.325 0)
+		(at 30.48 68.58 0)
 		(unit 1)
 		(exclude_from_sim no)
@@
 		(fields_autoplaced yes)
 		(property "Reference" "#PWR061"
-			(at 30.48 66.675 0)
+			(at 30.48 74.93 0)
 			(effects
 				(font
@@
 		)
 		(property "Value" "GND"
-			(at 30.48 65.405 0)
+			(at 30.48 73.66 0)
 			(effects
 				(font
@@
 		)
 		(property "Footprint" ""
-			(at 30.48 60.325 0)
+			(at 30.48 68.58 0)
 			(effects
 				(font
@@
 		)
 		(property "Datasheet" ""
-			(at 30.48 60.325 0)
+			(at 30.48 68.58 0)
 			(effects
 				(font
@@
 		)
 		(property "Description" ""
-			(at 30.48 60.325 0)
+			(at 30.48 68.58 0)
 			(effects
 				(font

Commit message: New pcb 3
Full connections and logotypes
Parts:
- D5, D6, D7: footprint Diode_SMD:D_1206_3216Metric -> LED_SMD:LED_1206_3216Metric
- R23, R24, R29, R30, R32, R33, R34, R35, R36, R37, R38, R39, R40, R41, R42, R43: footprint LED_SMD:LED_1206_3216Metric -> Resistor_SMD:R_1206_3216Metric
Changed lines of the file:
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@@
 			)
 		)
-		(property "Footprint" "LED_SMD:LED_1206_3216Metric"
+		(property "Footprint" "Resistor_SMD:R_1206_3216Metric"
 			(at 32.639 98.806 90)
 			(effects
@@
 			)
 		)
-		(property "Footprint" "Diode_SMD:D_1206_3216Metric"
+		(property "Footprint" "LED_SMD:LED_1206_3216Metric"
 			(at 155.194 177.927 0)
 			(effects
@@
 			)
 		)
-		(property "Footprint" "LED_SMD:LED_1206_3216Metric"
+		(property "Footprint" "Resistor_SMD:R_1206_3216Metric"
 			(at 121.539 113.284 90)
 			(effects
@@
 			)
 		)
-		(property "Footprint" "LED_SMD:LED_1206_3216Metric"
+		(property "Footprint" "Resistor_SMD:R_1206_3216Metric"
 			(at 128.016 185.547 90)
 			(effects
@@
 			)
 		)
-		(property "Footprint" "LED_SMD:LED_1206_3216Metric"
+		(property "Footprint" "Resistor_SMD:R_1206_3216Metric"
 			(at 204.343 146.685 90)
 			(effects
@@
 			)
 		)
-		(property "Footprint" "LED_SMD:LED_1206_3216Metric"
+		(property "Footprint" "Resistor_SMD:R_1206_3216Metric"
 			(at 153.416 185.547 90)
 			(effects
@@
 			)
 		)
-		(property "Footprint" "LED_SMD:LED_1206_3216Metric"
+		(property "Footprint" "Resistor_SMD:R_1206_3216Metric"
 			(at 63.373 188.595 90)
 			(effects
@@
 			)
 		)
-		(property "Footprint" "LED_SMD:LED_1206_3216Metric"
+		(property "Footprint" "Resistor_SMD:R_1206_3216Metric"
 			(at 194.31 90.932 90)
 			(effects
@@
 			)
 		)
-		(property "Footprint" "Diode_SMD:D_1206_3216Metric"
+		(property "Footprint" "LED_SMD:LED_1206_3216Metric"
 			(at 129.794 177.927 0)
 			(effects
@@
 			)
 		)
-		(property "Footprint" "LED_SMD:LED_1206_3216Metric"
+		(property "Footprint" "Resistor_SMD:R_1206_3216Metric"
 			(at 140.716 185.547 90)
 			(effects
@@
 			)
 		)
-		(property "Footprint" "Diode_SMD:D_1206_3216Metric"
+		(property "Footprint" "LED_SMD:LED_1206_3216Metric"
 			(at 142.494 177.927 0)
 			(effects
@@
 			)
 		)
-		(property "Footprint" "LED_SMD:LED_1206_3216Metric"
+		(property "Footprint" "Resistor_SMD:R_1206_3216Metric"
 			(at 32.639 106.426 90)
 			(effects
@@
 			)
 		)
-		(property "Footprint" "LED_SMD:LED_1206_3216Metric"
+		(property "Footprint" "Resistor_SMD:R_1206_3216Metric"
 			(at 63.373 170.815 90)
 			(effects
@@
 			)
 		)
-		(property "Footprint" "LED_SMD:LED_1206_3216Metric"
+		(property "Footprint" "Resistor_SMD:R_1206_3216Metric"
 			(at 193.675 139.827 90)
 			(effects
@@
 			)
 		)
-		(property "Footprint" "LED_SMD:LED_1206_3216Metric"
+		(property "Footprint" "Resistor_SMD:R_1206_3216Metric"
 			(at 204.343 51.435 90)
 			(effects
@@
 			)
 		)
-		(property "Footprint" "LED_SMD:LED_1206_3216Metric"
+		(property "Footprint" "Resistor_SMD:R_1206_3216Metric"
 			(at 124.079 90.932 90)
 			(effects
@@
 			)
 		)
-		(property "Footprint" "LED_SMD:LED_1206_3216Metric"
+		(property "Footprint" "Resistor_SMD:R_1206_3216Metric"
 			(at 120.523 52.705 90)
 			(effects
@@
 			)
 		)
-		(property "Footprint" "LED_SMD:LED_1206_3216Metric"
+		(property "Footprint" "Resistor_SMD:R_1206_3216Metric"
 			(at 193.675 44.577 90)
 			(effects
@@
 			)
 		)
-		(property "Footprint" "LED_SMD:LED_1206_3216Metric"
+		(property "Footprint" "Resistor_SMD:R_1206_3216Metric"
 			(at 204.978 97.79 90)
 			(effects
