File: schematic-main.kicad_sch (KiCad schematic)
At the start: 12 parts, among them J1 Fell_Cell_IN, J2 CAN, J3 P_Valve, J4 FC Cooling, J5 Valve, J7 Axilary_Out, J9 Analog_In, P1 USB_C_Plug_USB2.0

Commit message: P1
Parts:
- J2: symbol Connector_Generic:Conn_01x02 -> Connector_Generic:Conn_01x03
Connections:
- net GND: now also J2.3 (Pin_3)
Changed lines of the file:
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@@
     (stroke (width 0) (type default))
   )
-  (wire (pts (xy 63.6016 40.6654) (xy 63.6016 111.76))
+  (wire (pts (xy 62.23 40.64) (xy 62.23 111.76))
     (stroke (width 0) (type default))
   )
@@
     (stroke (width 0) (type default))
   )
-  (wire (pts (xy 126.492 119.634) (xy 134.62 119.634))
+  (wire (pts (xy 126.365 119.38) (xy 134.62 119.38))
     (stroke (width 0) (type default))
   )
@@
     (stroke (width 0) (type default))
   )
-  (wire (pts (xy 63.6016 111.76) (xy 134.62 111.76))
+  (wire (pts (xy 62.23 111.76) (xy 134.62 111.76))
     (stroke (width 0) (type default))
   )
@@
     (stroke (width 0) (type default))
   )
-  (wire (pts (xy 126.492 122.174) (xy 134.62 122.174))
+  (wire (pts (xy 126.365 121.92) (xy 134.62 121.92))
     (stroke (width 0) (type default))
   )
@@
         (path "/c9ad7189-d3b2-414a-9743-efd8e57cd755"
           (reference "#PWR055") (unit 1)
+        )
+      )
+    )
+  )
+  (symbol (lib_id "power:GND") (at 126.365 124.46 0) (unit 1)
+    (in_bom yes) (on_board yes) (dnp no) (fields_autoplaced)
+    (property "Reference" "#PWR089" (at 126.365 130.81 0)
+      (effects (font (size 1.27 1.27)) hide)
+    )
+    (property "Value" "GND" (at 126.365 129.54 0)
+      (effects (font (size 1.27 1.27)) hide)
+    )
+    (property "Footprint" "" (at 126.365 124.46 0)
+      (effects (font (size 1.27 1.27)) hide)
+    )
+    (property "Datasheet" "" (at 126.365 124.46 0)
+      (effects (font (size 1.27 1.27)) hide)
+    )
+    (pin "1")
+    (instances
+      (project "schematic-main"
+        (path "/c9ad7189-d3b2-414a-9743-efd8e57cd755"
+          (reference "#PWR089") (unit 1)
         )
       )
@@
     )
   )
-  (symbol (lib_id "power:+12V") (at 63.6016 40.6654 0) (unit 1)
-    (in_bom yes) (on_board yes) (dnp no) (fields_autoplaced)
-    (property "Reference" "#PWR070" (at 63.6016 44.4754 0)
-      (effects (font (size 1.27 1.27)) hide)
-    )
-    (property "Value" "+12V" (at 63.6016 35.5854 0)
-      (effects (font (size 1.27 1.27)))
-    )
-    (property "Footprint" "" (at 63.6016 40.6654 0)
-      (effects (font (size 1.27 1.27)) hide)
-    )
-    (property "Datasheet" "" (at 63.6016 40.6654 0)
+  (symbol (lib_id "power:+12V") (at 62.23 40.64 0) (unit 1)
+    (in_bom yes) (on_board yes) (dnp no) (fields_autoplaced)
+    (property "Reference" "#PWR070" (at 62.23 44.45 0)
+      (effects (font (size 1.27 1.27)) hide)
+    )
+    (property "Value" "+12V" (at 62.23 35.56 0)
+      (effects (font (size 1.27 1.27)))
+    )
+    (property "Footprint" "" (at 62.23 40.64 0)
+      (effects (font (size 1.27 1.27)) hide)
+    )
+    (property "Datasheet" "" (at 62.23 40.64 0)
       (effects (font (size 1.27 1.27)) hide)
     )
@@
     )
   )
-  (symbol (lib_id "Connector_Generic:Conn_01x02") (at 121.412 119.634 0) (mirror y) (unit 1)
+  (symbol (lib_id "Connector_Generic:Conn_01x03") (at 121.285 121.92 0) (mirror y) (unit 1)
     (in_bom yes) (on_board yes) (dnp no)
-    (property "Reference" "J2" (at 118.872 119.634 0)
-      (effects (font (size 1.27 1.27)) (justify left))
-    )
-    (property "Value" "CAN" (at 118.872 122.174 0)
-      (effects (font (size 1.27 1.27)) (justify left))
-    )
-    (property "Footprint" "Connector_Molex:Molex_Mini-Fit_Jr_5569-02A2_2x01_P4.20mm_Horizontal" (at 121.412 119.634 0)
-      (effects (font (size 1.27 1.27)) hide)
-    )
-    (property "Datasheet" "~" (at 121.412 119.634 0)
-      (effects (font (size 1.27 1.27)) hide)
-    )
-    (pin "1")
-    (pin "2")
+    (property "Reference" "J2" (at 118.745 121.92 0)
+      (effects (font (size 1.27 1.27)) (justify left))
+    )
+    (property "Value" "CAN" (at 118.745 124.46 0)
+      (effects (font (size 1.27 1.27)) (justify left))
+    )
+    (property "Footprint" "Connector_Molex:Molex_Mini-Fit_Jr_5569-02A2_2x01_P4.20mm_Horizontal" (at 121.285 121.92 0)
+      (effects (font (size 1.27 1.27)) hide)
+    )
+    (property "Datasheet" "~" (at 121.285 121.92 0)
+      (effects (font (size 1.27 1.27)) hide)
+    )
+    (pin "1")
+    (pin "2")
+    (pin "3")
     (instances
       (project "schematic-main"
@@
       (effects (font (size 1.27 1.27)) (justify right))
     )
-    (pin "CANH" bidirectional (at 134.62 119.634 180)
-      (effects (font (size 1.27 1.27)) (justify left))
-    )
-    (pin "CANL" bidirectional (at 134.62 122.174 180)
-      (effects (font (size 1.27 1.27)) (justify left))
-    )
+    (pin "CANH" bidirectional (at 134.62 119.38 180)
+      (effects (font (size 1.27 1.27)) (justify left))
+    )
+    (pin "CANL" bidirectional (at 134.62 121.92 180)
+      (effects (font (size 1.27 1.27)) (justify left))
+    )

Commit message: Edit main
Changed lines of the file:
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@@
   (junction (at 93.98 85.09) (diameter 0) (color 0 0 0 0)
   )
-  (junction (at 31.75 31.75) (diameter 0) (color 0 0 0 0)
-  )
   (junction (at 73.66 33.02) (diameter 0) (color 0 0 0 0)
   )
@@
     (stroke (width 0) (type default))
   )
-  (wire (pts (xy 29.21 31.75) (xy 31.75 31.75))
-    (stroke (width 0) (type default))
-  )
   (wire (pts (xy 102.87 85.09) (xy 111.76 85.09))
     (stroke (width 0) (type default))
@@
     (stroke (width 0) (type default))
   )
-  (wire (pts (xy 31.75 31.75) (xy 46.99 31.75))
+  (wire (pts (xy 29.21 31.75) (xy 46.99 31.75))
     (stroke (width 0) (type default))
   )
@@
         )
       )
-    )
-  )
-  (symbol (lib_id "power:PWR_FLAG") (at 31.75 31.75 0) (unit 1)
-    (in_bom yes) (on_board yes) (dnp no)
-    (property "Reference" "#FLG01" (at 31.75 29.845 0)
-      (effects (font (size 1.27 1.27)) hide)
-    )
-    (property "Value" "PWR_FLAG" (at 26.67 26.67 0)
-      (effects (font (size 1.27 1.27)) (justify left))
-    )
-    (property "Footprint" "" (at 31.75 31.75 0)
-      (effects (font (size 1.27 1.27)) hide)
-    )
-    (property "Datasheet" "~" (at 31.75 31.75 0)
-      (effects (font (size 1.27 1.27)) hide)
-    )
-    (pin "1")
-    (instances
-      (project "schematic-main"
-        (path "/c9ad7189-d3b2-414a-9743-efd8e57cd755"
-          (reference "#FLG01") (unit 1)
-        )
-      )

Commit message: New pcb 1
Parts:
- J3: renamed from J2; footprint Connector_Molex:Molex_Mini-Fit_Jr_5569-02A2_2x01_P4.20mm_Horizontal -> library:39303035
- renumbered J9 to J2, J7 to J4, J3 to J5, J5 to J6, J4 to J7, R3 to R1, R1 to R2, R2 to R3

Commit message: New pcb 2
Near complate
Connections:
- net IO/FAN_PWM renamed IO/FAN_IN_PWM
Other:
- sheet IO ports: added 5V, FAN_IN_PWM, FAN_IN_PWM_MCU, FC_V, I/O_1_MCU, I/O_2_MCU, I/O_3_MCU, I/O_4_MCU; removed FAN_PWM, SC_V
- sheet MCU ports: added FAN_IN_PWM_MCU, I/O_1_MCU, I/O_2_MCU, I/O_3_MCU, I/O_4_MCU; removed none
- sheet Power  ports: added FC_V; removed SC_V

Commit message: New pcb 3
Full connections and logotypes
Other:
- sheet IO ports: added none; removed FAN_PWM_MCU
- sheet MCU ports: added none; removed FAN_PWM_MCU
Changed lines of the file:
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@@
-	(wire
-		(pts
-			(xy 179.959 81.28) (xy 179.959 104.14)
-		)
-		(stroke
-			(width 0)
-			(type default)
-		)
-	)
 	(wire
 		(pts
@@
 			)
 		)
-		(pin "FAN_PWM_MCU" input
-			(at 179.959 104.14 90)
-			(effects
-				(font
-					(size 1.27 1.27)
-				)
-				(justify right)
-			)
-		)
 		(pin "PURGE_VALVE_MCU" input
 			(at 182.499 104.14 90)
@@
 			(effects
 				(font
-					(size 1.27 1.27)
-				)
-				(justify left)
-			)
-		)
-		(pin "FAN_PWM_MCU" output
-			(at 179.959 81.28 270)
-			(effects
-				(font
