File: schematic-mcu.kicad_sch (KiCad schematic)
At the start: 28 parts, among them U3 USBLC6-2P6, U4 ESP32-S3FN8, Y1 Crystal_GND24

Commit message: New pcb 2
Near complate
Parts:
- added R47, R48: 10k, LED_SMD:LED_1206_3216Metric, symbol Device:R
Connections:
- net +3.3V: now also R48.2
- net GND: now also R47.2
- net FAN_IN_PWM_MCU: now reaches U4.51 (GPIO45)
- net FAN_IN_PWM_MCU: now also R47.1, R48.1
- no-connect marks 26 -> 25

Commit message: New pcb 3
Full connections and logotypes
Parts:
- removed R21: 10k, LED_SMD:LED_1206_3216Metric, symbol Device:R
- R18, R19, R20, R22, R47, R48: footprint LED_SMD:LED_1206_3216Metric -> Resistor_SMD:R_1206_3216Metric
Connections:
- net FAN_PWM_MCU: no longer names the net of U4.28 (SPI_CS1/GPIO26)
Changed lines of the file:
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@@
 		(color 0 0 0 0)
 	)
-	(junction
-		(at 172.847 110.236)
-		(diameter 0)
-		(color 0 0 0 0)
-	)
 	(no_connect
 		(at 261.62 77.47)
@@
 	(wire
 		(pts
-			(xy 172.847 110.236) (xy 176.911 110.236)
-		)
-		(stroke
-			(width 0)
-			(type default)
-		)
-	)
-	(wire
-		(pts
-			(xy 176.911 110.236) (xy 176.911 118.11)
-		)
-		(stroke
-			(width 0)
-			(type default)
-		)
-	)
-	(wire
-		(pts
 			(xy 191.77 135.89) (xy 195.58 135.89)
 		)
@@
 	(wire
 		(pts
-			(xy 166.497 110.236) (xy 172.847 110.236)
-		)
-		(stroke
-			(width 0)
-			(type default)
-		)
-	)
-	(wire
-		(pts
 			(xy 203.2 53.34) (xy 219.71 53.34)
 		)
@@
 	(wire
 		(pts
-			(xy 176.911 118.11) (xy 195.58 118.11)
-		)
-		(stroke
-			(width 0)
-			(type default)
-		)
-	)
-	(wire
-		(pts
 			(xy 45.339 159.639) (xy 45.339 149.479)
 		)
@@
 	(wire
 		(pts
-			(xy 169.037 102.616) (xy 172.847 102.616)
-		)
-		(stroke
-			(width 0)
-			(type default)
-		)
-	)
-	(wire
-		(pts
 			(xy 43.18 40.64) (xy 43.18 41.91)
 		)
@@
 		)
 	)
-	(hierarchical_label "FAN_PWM_MCU"
-		(shape output)
-		(at 166.497 110.236 180)
-		(fields_autoplaced yes)
-		(effects
-			(font
-				(size 1.27 1.27)
-			)
-			(justify right)
-		)
-	)
 	(hierarchical_label "FC_Voltage_MCU"
 		(shape input)
@@
 			)
 		)
-		(property "Footprint" "LED_SMD:LED_1206_3216Metric"
+		(property "Footprint" "Resistor_SMD:R_1206_3216Metric"
 			(at 267.208 134.62 90)
 			(effects
@@
 			)
 		)
-		(property "Footprint" "LED_SMD:LED_1206_3216Metric"
+		(property "Footprint" "Resistor_SMD:R_1206_3216Metric"
 			(at 124.968 36.83 90)
 			(effects
@@
 	(symbol
 		(lib_id "power:GND")
-		(at 169.037 102.616 0)
-		(unit 1)
-		(exclude_from_sim no)
-		(in_bom yes)
-		(on_board yes)
-		(dnp no)
-		(fields_autoplaced yes)
-		(property "Reference" "#PWR046"
-			(at 169.037 108.966 0)
-			(effects
-				(font
-					(size 1.27 1.27)
-				)
-				(hide yes)
-			)
-		)
-		(property "Value" "GND"
-			(at 169.037 107.696 0)
-			(effects
-				(font
-					(size 1.27 1.27)
-				)
-				(hide yes)
-			)
-		)
-		(property "Footprint" ""
-			(at 169.037 102.616 0)
-			(effects
-				(font
-					(size 1.27 1.27)
-				)
-				(hide yes)
-			)
-		)
-		(property "Datasheet" ""
-			(at 169.037 102.616 0)
-			(effects
-				(font
-					(size 1.27 1.27)
-				)
-				(hide yes)
-			)
-		)
-		(property "Description" ""
-			(at 169.037 102.616 0)
-			(effects
-				(font
-					(size 1.27 1.27)
-				)
-				(hide yes)
-			)
-		)
-		(pin "1"
-		)
-		(instances
-			(project "schematic-main"
-				(path "/c9ad7189-d3b2-414a-9743-efd8e57cd755/f92f58ec-64e0-437c-bc00-8ae46a3b3054"
-					(reference "#PWR046")
-					(unit 1)
-				)
-			)
-		)
-	)
-	(symbol
-		(lib_id "power:GND")
 		(at 256.54 66.04 0)
 		(unit 1)
@@
 	)
 	(symbol
-		(lib_id "Device:R")
-		(at 172.847 106.426 180)
-		(unit 1)
-		(exclude_from_sim no)
-		(in_bom yes)
-		(on_board yes)
-		(dnp no)
-		(fields_autoplaced yes)
-		(property "Reference" "R21"
-			(at 174.752 105.1559 0)
-			(effects
-				(font
-					(size 1.27 1.27)
-				)
-				(justify right)
-			)
-		)
-		(property "Value" "10k"
-			(at 174.752 107.6959 0)
-			(effects
-				(font
-					(size 1.27 1.27)
-				)
-				(justify right)
-			)
-		)
-		(property "Footprint" "LED_SMD:LED_1206_3216Metric"
-			(at 174.625 106.426 90)
-			(effects
-				(font
-					(size 1.27 1.27)
-				)
-				(hide yes)
-			)
-		)
-		(property "Datasheet" "~"
-			(at 172.847 106.426 0)
-			(effects
-				(font
-					(size 1.27 1.27)
-				)
-				(hide yes)
-			)
-		)
-		(property "Description" ""
-			(at 172.847 106.426 0)
-			(effects
-				(font
-					(size 1.27 1.27)
-				)
-				(hide yes)
-			)
-		)
-		(pin "1"
-		)
-		(pin "2"
-		)
-		(instances
-			(project "schematic-main"
-				(path "/c9ad7189-d3b2-414a-9743-efd8e57cd755/f92f58ec-64e0-437c-bc00-8ae46a3b3054"
-					(reference "R21")
-					(unit 1)
-				)
-			)
-		)
-	)
-	(symbol
 		(lib_id "power:+3.3V")
 		(at 43.18 31.75 0)
@@
 			)
 		)
-		(property "Footprint" "LED_SMD:LED_1206_3216Metric"
+		(property "Footprint" "Resistor_SMD:R_1206_3216Metric"
 			(at 184.15 158.623 90)
 			(effects
@@
 			)
 		)
-		(property "Footprint" "LED_SMD:LED_1206_3216Metric"
+		(property "Footprint" "Resistor_SMD:R_1206_3216Metric"
 			(at 143.129 122.174 90)
 			(effects
@@
 			)
 		)
-		(property "Footprint" "LED_SMD:LED_1206_3216Metric"
+		(property "Footprint" "Resistor_SMD:R_1206_3216Metric"
 			(at 137.16 141.224 90)
 			(effects
@@
 			)
 		)
-		(property "Footprint" "LED_SMD:LED_1206_3216Metric"
+		(property "Footprint" "Resistor_SMD:R_1206_3216Metric"
 			(at 263.652 142.24 90)
 			(effects
