File: schematic-power.kicad_sch (KiCad schematic)
At the start: 36 parts, among them IC2 LM76202QPWPRQ1, U6 LM5013DDAR, U9 TPS62933

Commit message: New pcb 1
Parts:
- removed F2: 3A, mbr:FUSC8664X180N, symbol Device:Fuse
- F1: footprint mbr:FUSC8664X180N -> library:FUSC8664X180N
- IC1: renamed from IC2; footprint mbr:SOP65P640X120-17N -> library:SOP65P640X120-17N
- TP1: footprint (none) -> Connector_PinSocket_2.54mm:PinSocket_1x01_P2.54mm_Vertical
- renumbered C26 to C1, C28 to C3, C29 to C5, C30 to C6, C27 to C8, D7 to D2, D2 to D3, L3 to L1, R15 to R10, R24 to R12, R25 to R13, R14 to R5, U6 to U1
Connections:
- net +12V: now also C6.2, C8.1, L1.2, R12.2
Other:
- moved on the sheet: C8

Commit message: Power stage pcb complate
Connections:
- net SC_V renamed FC_V

Commit message: New pcb 3
Full connections and logotypes
Parts:
- R12, R13: footprint LED_SMD:LED_1206_3216Metric -> Resistor_SMD:R_1206_3216Metric
Changed lines of the file:
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@@
 			)
 		)
-		(property "Footprint" "LED_SMD:LED_1206_3216Metric"
+		(property "Footprint" "Resistor_SMD:R_1206_3216Metric"
 			(at 142.875 73.66 90)
 			(effects
@@
 			)
 		)
-		(property "Footprint" "LED_SMD:LED_1206_3216Metric"
+		(property "Footprint" "Resistor_SMD:R_1206_3216Metric"
 			(at 142.875 66.04 90)
 			(effects
