File: schematic-main.kicad_pcb (KiCad board)
At the start: 2 copper layers, 100 x 100 mm, 132 parts, among them IC1 LM76202QPWPRQ1, IC2 AD8544ARUZ-REEL, J1 Fell_Cell_IN, J2 Analog_In, J3 CAN, J4 Axilary_Out, J5 P_Valve, J6 Valve, J7 FC Cooling, P1 USB_C_Plug_USB2.0, Q1 PMPB10XNX, Q2 PMPB10XNX, Q3 PMPB10XNX, U1 LM5013DDAR, U2 TPS62933, U3 USBLC6-2P6, U4 ESP32-S3FN8, U5 SN65HVD232, Y1 Crystal_GND24

Commit message: New pcb 2
Near complate
Parts:
- added R47: 10k, LED_SMD:LED_1206_3216Metric, F.Cu at (134.4, 80.8)
- added R48: 10k, LED_SMD:LED_1206_3216Metric, F.Cu at (128.6, 80.7)
- moved L3 142.3 mm to (110.5, 83.7), turned to -90 degrees
- moved R37 137.8 mm to (135.5, 56.5), turned to 90 degrees
- moved C23 136.7 mm to (107.7, 84.6), turned to -90 degrees
- moved C22 136.5 mm to (107.9, 79.6), turned to 90 degrees
- moved C27 134.8 mm to (110.4, 79.6), turned to 90 degrees
- moved C24 132.8 mm to (111.6, 85.9), turned to 180 degrees
- moved R36 126.4 mm to (134.7, 89.8)
- moved R35 126.4 mm to (134.8, 85.9)
- moved C25 125.8 mm to (118.8, 95.1), turned to -90 degrees
- moved R21 125.1 mm to (126.6, 97.6), turned to -90 degrees
- moved C26 121.2 mm to (123.7, 80.7), turned to 90 degrees
- moved R22 118.8 mm to (131.6, 71.3)
- moved R42 111.1 mm to (161.2, 78.9), turned to -90 degrees
- moved R39 110.2 mm to (159.7, 75.0), turned to 180 degrees
- moved R38 106.3 mm to (150.8, 85.1), turned to 180 degrees
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Connections:
- C1 pad 1: /Power /SC_V -> /IO/FC_V
- D3 pad 1: /VBUS -> +5V
- F1 pad 2: /Power /SC_V -> /IO/FC_V
- J7 pad 2: /FAN_PWM -> /IO/FAN_IN_PWM
- J7 pad 7: /FAN_PWM -> /IO/FAN_IN_PWM
- P1 pad A4: /VBUS -> +5V
- P1 pad A9: /VBUS -> +5V
- P1 pad B4: /VBUS -> +5V
- P1 pad B9: /VBUS -> +5V
- TP1 pad 1: /Power /SC_V -> /IO/FC_V
- U1 pad 2: /Power /SC_V -> /IO/FC_V
- U1 pad 3: /Power /SC_V -> /IO/FC_V
- U4 pad 12: /MCU/I/O_1_MCU -> /IO/I/O_1_MCU
- U4 pad 13: /MCU/I/O_2_MCU -> /IO/I/O_2_MCU
- U4 pad 16: /MCU/I/O_3_MCU -> /IO/I/O_3_MCU
- U4 pad 18: /MCU/I/O_4_MCU -> /IO/I/O_4_MCU
- U4 pad 51: unconnected-(U4-GPIO45-Pad51) -> /IO/FAN_IN_PWM
Routing:
- net GND: track 371.1 -> 803.0 mm, vias 35 -> 80
- net +3.3V: track 71.0 -> 384.5 mm, vias 1 -> 11
- net +12V: track 61.8 -> 352.3 mm, vias 0 -> 10
- net +5V: track 0.00 -> 163.0 mm, vias 0 -> 3
- net /VBUS: track 157.4 -> 0.00 mm, vias 3 -> 0
- net /IO/A_Input: track 11.8 -> 149.2 mm
- net /IO/FAN_1_TACHO: track 2.83 -> 64.5 mm, vias 0 -> 2
- net /IO/FC_Voltage_MCU: track 92.1 -> 34.8 mm, vias 1 -> 2
- net /IO/FAN_2_TACHO: track 0.78 -> 55.4 mm, vias 0 -> 2
- net /IO/FAN_IN_PWM: track 0.00 -> 54.2 mm, vias 0 -> 2
- net /IO/FC_V: track 2.04 -> 56.2 mm
- net /IO/PURGE_VALVE: track 0.00 -> 51.9 mm
- net /IO/Main_Valve: track 0.00 -> 41.4 mm
- net /IO/FAN_ON_MCU: track 0.00 -> 39.6 mm, vias 0 -> 2
- net /IO/CAN_TX: track 0.00 -> 39.3 mm, vias 0 -> 1
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Other:
- outline, holes or cut-outs redrawn

Commit message: New pcb 3
Full connections and logotypes
Parts:
- removed R21: 10k, LED_SMD:LED_1206_3216Metric
- D5, D6, D7: footprint Diode_SMD:D_1206_3216Metric -> LED_SMD:LED_1206_3216Metric
- R12, R13, R18, R19, R20, R22, R23, R24, R29, R30, R32, R33, R34, R35, R36, R37, R38, R39, R40, R41, R42, R43, R47, R48: footprint LED_SMD:LED_1206_3216Metric -> Resistor_SMD:R_1206_3216Metric
- moved TP8 65.1 mm to (161.4, 100.0), turned to 180 degrees
- moved TP9 60.4 mm to (156.4, 100.0), turned to 180 degrees
- moved R38 6.98 mm to (157.8, 85.3), turned to -90 degrees
- moved R44 3.32 mm to (182.6, 92.4)
- moved C35 2.64 mm to (175.6, 93.4)
- moved D6 2.62 mm to (132.0, 89.0)
- moved R36 2.62 mm to (137.2, 89.0)
- moved TP12 2.43 mm to (102.2, 98.6)
- moved D5 2.40 mm to (131.9, 85.9)
- moved R35 2.40 mm to (137.2, 85.9)
- moved TP13 1.81 mm to (106.2, 101.1)
- moved R37 1.47 mm to (135.7, 55.0), turned to 0 degrees
- moved TP2 1.39 mm to (96.2, 75.0)
- moved TP3 1.39 mm to (101.2, 75.0)
- moved R19 1.30 mm to (165.7, 67.6)
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Connections:
- U4 pad 28: /MCU/FAN_PWM_MCU -> unconnected-(U4-SPI_CS1/GPIO26-Pad28)
Routing:
- net GND: track 803.0 -> 998.1 mm, vias 80 -> 212
- net +3.3V: track 384.5 -> 516.8 mm, vias 11 -> 15
- net /IO/Temp_MCU: track 7.27 -> 87.3 mm
- net /MCU/MCU_TEST: track 10.8 -> 69.8 mm, vias 1 -> 2
- net +12V: track 352.3 -> 314.9 mm, vias 10 -> 14
- net /IO/Analog_MCU: track 42.6 -> 79.6 mm
- net /IO/FC_Voltage_MCU: track 34.8 -> 66.6 mm
- net /MCU/BOOT: track 14.5 -> 44.1 mm, vias 1 -> 2
- net /MCU/RESET: track 13.8 -> 42.8 mm, vias 1 -> 2
- net /IO/CAN_RX: track 16.4 -> 39.0 mm
- net /IO/FAN_GND: track 26.2 -> 46.4 mm
- net /MCU/USB_D-: track 9.33 -> 29.0 mm, vias 1 -> 0
- net /IO/FAN_IN_PWM: track 54.2 -> 71.8 mm, vias 2 -> 3
- net /MCU/USB_D+: track 9.11 -> 26.1 mm, vias 1 -> 0
- net /IO/FAN_2_TACHO: track 55.4 -> 68.3 mm
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Other:
- board text added: "Fuel Cell Unit v1 Michał Borkowski 05.03.2024"

Commit message: New pcb 4
Parts:
- renumbered TP10 to TP1, TP11 to TP2
Other:
- board text added: "+12V GND"
- board text added: "+12V Main_Valve_G"
- board text added: "+3,3V A_Input"
- board text added: "2x +12V"
- board text added: "2x +12V 2x Fan_IN_PWM"
- board text added: "2x +3,3V"
- board text added: "2x +5V USB"
- board text added: "2x FAN_G +3,3V Temp_sensor"
- board text added: "2x GND"
- board text added: "CAN: H L GND"
- board text added: "FC_test"
- board text added: "GND Fuel_Cell+"
- board text added: "I/O 1 I/O 2"
- board text added: "I/O 3 I/O 4"
- board text added: "MCU_TEST"
- board text added: "Purge_Valve_G +12V"
- board text added: "RESET BOOT"
- board text added: "Tacho 2 1"

Commit message: New pcb 5
Routing:
- net Net-(D2-K): vias 2 -> 3
Other:
- board text added: "+12V"
- board text added: "+3.3V"
- board text added: "+Fuel cell"
- board text added: "Analog input"
- board text added: "CAN"
- board text added: "CAN High"
- board text added: "CAN Low"
- board text added: "FC Power"
- board text added: "Fan 1 tacho"
- board text added: "Fan 2 tacho"
- board text added: "Fan GND"
- board text added: "Fan PWM"
- board text added: "Fuel cell"
- board text added: "GND"
- board text added: "Main valve GND"
- board text added: "Purge valve GND"
- board text added: "Temp sensor"
