File: schematic-main.kicad_pcb (KiCad board)
At the start: 2 copper layers, 100 x 100 mm, 133 parts, among them IC1 LM76202QPWPRQ1, IC2 AD8544ARUZ-REEL, J1 Fell_Cell_IN, J2 Analog_In, J3 CAN, J4 Axilary_Out, J5 P_Valve, J6 Valve, J7 FC Cooling, P1 USB_C_Plug_USB2.0, Q1 PMPB10XNX, Q2 PMPB10XNX, Q3 PMPB10XNX, U1 LM5013DDAR, U2 TPS62933, U3 USBLC6-2P6, U4 ESP32-S3FN8, U5 SN65HVD232, Y1 Crystal_GND24

Commit message: New pcb 6 end
Parts:
- added REF**: MountingHole_3mm, MountingHole:MountingHole_3mm, F.Cu at (98.5, 20.5)
- added REF**: MountingHole_3mm, MountingHole:MountingHole_3mm, F.Cu at (185.0, 21.0)
- added REF**: MountingHole_3mm, MountingHole:MountingHole_3mm, F.Cu at (162.3, 109.3)
Routing:
- net Net-(D2-K): vias 3 -> 2
- net GND: vias 212 -> 210
Other:
- outline, holes or cut-outs redrawn

Commit message: DRC tested
Parts:
- D5 CAN: renamed from D5
- D6 MCU: renamed from D6
- D7 POWER 3.3V: renamed from D7
Routing:
- net /Power /Vreg: track 32.1 -> 45.1 mm
- net +5V: track 161.1 -> 165.4 mm
- net +3.3V: track 516.8 -> 515.3 mm
- net Net-(U2-VIN): track 58.9 -> 59.8 mm
Other:
- board text added: "2x +3.3V"
- board text removed: "2x +3,3V"
